Commit message: 9주차 과제

File: urdf_tutorial/urdf/01-myfirst.urdf (robot description, URDF)
Before this commit: robot testbot, 5 links, 4 joints
Links:
- removed link base
- removed link link1
- removed link link2
- removed link link3
- removed link link4
- added link base_link; visual cylinder length=0.6 radius=0.2
Joints:
- removed joint fixed
- removed joint joint1
- removed joint joint2
- removed joint link3
